Commit message: tweak labyrinth environment

File: two_blocks/two_blocks_env/assets/labyrinth.urdf (robot description, URDF)
Before this commit: robot tomas-labyrinth, 5 links, 4 joints
Links:
- link left_wall: geometry collision box size=20 0.5 1.5; visual box size=20 0.5 1.5
- link middle_wall: geometry collision box size=16 0.5 1.5; visual box size=16 0.5 1.5
- link north_wall: geometry collision box size=10 0.5 1.5; visual box size=10 0.5 1.5
- link right_wall: geometry collision box size=20 0.5 1.5; visual box size=20 0.5 1.5
- link south_wall: geometry collision box size=10 0.5 1.5; visual box size=10 0.5 1.5
