Commit message: Convert Pybullet Labyrinth to xacro file

File: multi_goal/envs/assets/immaterial_ball.urdf (robot description, URDF)
Before this commit: robot immaterial_ball, 1 links, 0 joints
Links:
- link baseLink: mass None -> 1

File: multi_goal/envs/assets/labyrinth.urdf (robot description, URDF)
Before this commit: robot tomas-labyrinth, 5 links, 4 joints
Links:
- link left_wall: mass None -> 0.5
- link middle_wall: mass None -> 0.5; geometry collision box size=20 0.5 1.5; visual box size=16 0.5 1.5
- link north_wall: mass None -> 0.5; geometry collision box size=20 0.5 1.5; visual box size=10 0.5 1.5
- link right_wall: mass None -> 0.5
- link south_wall: mass None -> 0.5; geometry collision box size=20 0.5 1.5; visual box size=10 0.5 1.5
