Commit message: Reduce wall thickness

File: multi_goal/envs/assets/labyrinth.urdf (robot description, URDF)
Before this commit: robot tomas-labyrinth, 5 links, 4 joints
Links:
- link left_wall: geometry collision box size=20 0.5 1.5; visual box size=20 0.31 1.5
- link middle_wall: geometry collision box size=20 0.5 1.5; visual box size=16 0.31 1.5
- link north_wall: geometry collision box size=20 0.5 1.5; visual box size=10 0.31 1.5
- link right_wall: geometry collision box size=20 0.5 1.5; visual box size=20 0.31 1.5
- link south_wall: geometry collision box size=20 0.5 1.5; visual box size=10 0.31 1.5

File: multi_goal/envs/assets/labyrinth.xacro (robot description, xacro)
@@ -8,5 +8,5 @@
       <visual>
         <geometry>
-          <box size="${length} 0.5 1.5"/>
+          <box size="${length} 0.31 1.5"/>
         </geometry>
         <material name="wall_color"/>

Commit message: Fix Labyrinth display/collision bug

File: multi_goal/envs/assets/labyrinth.urdf (robot description, URDF)
Before this commit: robot tomas-labyrinth, 5 links, 4 joints
Links:
- link left_wall: geometry collision box size=20 0.31 1.5; visual box size=20 0.31 1.5
- link middle_wall: geometry collision box size=16 0.31 1.5; visual box size=16 0.31 1.5
- link north_wall: geometry collision box size=10 0.31 1.5; visual box size=10 0.31 1.5
- link right_wall: geometry collision box size=20 0.31 1.5; visual box size=20 0.31 1.5
- link south_wall: geometry collision box size=10 0.31 1.5; visual box size=10 0.31 1.5

File: multi_goal/envs/assets/labyrinth.xacro (robot description, xacro)
@@ -14,5 +14,5 @@
       <collision>
         <geometry>
-          <box size="20 0.5 1.5"/>
+          <box size="${length} 0.31 1.5"/>
         </geometry>
       </collision>

Commit message: Add a harder PyBullet Labyrinth

File: multi_goal/envs/assets/labyrinth.urdf (robot description, URDF)
Before this commit: robot tomas-labyrinth, 5 links, 4 joints
Joints:
- removed joint wall_left_middle
- removed joint wall_left_north
- removed joint wall_left_right
- removed joint wall_left_south
- added joint left_wall-middle_wall: type fixed, parent left_wall, child middle_wall, origin xyz=-2 5 0 rpy=0 0 0
- added joint left_wall-north_wall: type fixed, parent left_wall, child north_wall, origin xyz=10 5 0 rpy=0 0 1.57079632679
- added joint left_wall-right_wall: type fixed, parent left_wall, child right_wall, origin xyz=0 10 0 rpy=0 0 0
- added joint left_wall-south_wall: type fixed, parent left_wall, child south_wall, origin xyz=-10 5 0 rpy=0 0 1.57079632679

File: multi_goal/envs/assets/labyrinth.xacro (robot description, xacro)
@@ -24,28 +24,19 @@
     </link>
   </xacro:macro>
+  <xacro:macro name="make_joint" params="parent child xyz rpy">
+    <joint name="${parent}-${child}" type="fixed">
+      <parent link="${parent}"/>
+      <child link="${child}"/>
+      <origin xyz="${xyz}" rpy="${rpy}"/>
+    </joint>
+  </xacro:macro>
   <xacro:make_wall name="left_wall" length="20"/>
   <xacro:make_wall name="right_wall" length="20"/>
-  <joint name="wall_left_right" type="fixed">
-    <parent link="left_wall"/>
-    <child link="right_wall"/>
-    <origin xyz="0 10 0"/>
-  </joint>
   <xacro:make_wall name="north_wall" length="10" />
   <xacro:make_wall name="south_wall" length="10" />
-  <joint name="wall_left_north" type="fixed">
-    <parent link="left_wall"/>
-    <child link="north_wall"/>
-    <origin xyz="10 5 0" rpy="0 0 1.57079"/>
-  </joint>
-  <joint name="wall_left_south" type="fixed">
-    <parent link="left_wall"/>
-    <child link="south_wall"/>
-    <origin xyz="-10 5 0" rpy="0 0 1.57079"/>
-  </joint>
   <xacro:make_wall name="middle_wall" length="16" />
-  <joint name="wall_left_middle" type="fixed">
-    <parent link="left_wall"/>
-    <child link="middle_wall"/>
-    <origin xyz="-2 5 0"/>
-  </joint>
+  <xacro:make_joint parent="left_wall" child="north_wall" xyz="10 5 0" rpy="0 0 ${pi/2}" />
+  <xacro:make_joint parent="left_wall" child="south_wall" xyz="-10 5 0" rpy="0 0 ${pi/2}" />
+  <xacro:make_joint parent="left_wall" child="middle_wall" xyz="-2 5 0" rpy="0 0 0" />
+  <xacro:make_joint parent="left_wall" child="right_wall" xyz="0 10 0" rpy="0 0 0" />
 </robot>
